File: hardware_design/Diode_Gate_1/Diode_Gate_1.kicad_pcb (KiCad board)
At the start: 2 copper layers, 32.5 x 10.2 mm, 4 parts, among them J1 Conn_Coaxial, J2 Conn_Coaxial

Commit message: added text, testing push
Other:
- board text added: "ARTS-Lab"
Changed lines of the file:
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@@
-(kicad_pcb (version 20171130) (host pcbnew "(5.1.5)-3")
+(kicad_pcb (version 20171130) (host pcbnew "(5.1.4)-1")
   (general
     (thickness 1.6)
-    (drawings 5)
+    (drawings 6)
     (tracks 10)
     (zones 0)
@@
   )
   (layers
-    (0 F.Cu signal)
+    (0 F.Cu signal hide)
     (31 B.Cu signal hide)
     (32 B.Adhes user)
@@
     )
   )
-  (gr_text "Diode Gate 1" (at 153.924 94.742) (layer B.SilkS)
+  (gr_text ARTS-Lab (at 154.051 98.4504) (layer B.SilkS)
+    (effects (font (size 1 1) (thickness 0.15)) (justify mirror))
+  )
+  (gr_text "Diode Gate 1" (at 154.1526 90.932) (layer B.SilkS)
     (effects (font (size 1.5 1.5) (thickness 0.3)) (justify mirror))
   )
