File: hardware_design/Diode_Gate_2/Diode_Gate_2.kicad_pcb (KiCad board)
At the start: 2 copper layers, 24.1 x 10.2 mm, 4 parts, among them J1 Conn_Coaxial, J2 Conn_Coaxial

Commit message: added text, testing push
Other:
- board text added: "Diode Gate 2 ARTS-Lab"
- board text removed: "Diode Gate 2"
Changed lines of the file:
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@@
-(kicad_pcb (version 20171130) (host pcbnew "(5.1.5)-3")
+(kicad_pcb (version 20171130) (host pcbnew "(5.1.4)-1")
   (general
     (thickness 1.6)
@@
   )
   (layers
-    (0 F.Cu signal)
-    (31 B.Cu signal)
+    (0 F.Cu signal hide)
+    (31 B.Cu signal hide)
     (32 B.Adhes user)
     (33 F.Adhes user)
@@
     )
   )
-  (gr_text "Diode Gate 2" (at 142.494 102.87) (layer B.SilkS)
+  (gr_text "Diode Gate 2\n ARTS-Lab" (at 142.621 103.2764) (layer B.SilkS)
     (effects (font (size 0.992 0.992) (thickness 0.1476)) (justify mirror))
   )
