File: hardware_design/Diode_Gate_3/Diode_Gate_3.kicad_pcb (KiCad board)
At the start: 2 copper layers, 33 x 10.7 mm, 7 parts, among them J1 Conn_Coaxial, J2 Conn_Coaxial

Commit message: added text, testing push
Other:
- board text added: "Diode Gate 3 ARTS-Lab"
Changed lines of the file:
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@@
-(kicad_pcb (version 20171130) (host pcbnew "(5.1.5)-3")
+(kicad_pcb (version 20171130) (host pcbnew "(5.1.4)-1")
   (general
     (thickness 1.6)
-    (drawings 4)
+    (drawings 5)
     (tracks 17)
     (zones 0)
@@
   )
   (setup
-    (last_trace_width 1.016)
+    (last_trace_width 0.1524)
     (user_trace_width 1.016)
     (trace_clearance 0.1524)
@@
     (solder_mask_min_width 0.25)
     (aux_axis_origin 0 0)
-    (visible_elements FFFFFF7F)
+    (visible_elements 7FFFFFFF)
     (pcbplotparams
       (layerselection 0x010fc_ffffffff)
@@
     )
   )
+  (gr_text "Diode Gate 3\n ARTS-Lab" (at 144.3482 102.3112) (layer B.SilkS)
+    (effects (font (size 1 1) (thickness 0.15)) (justify mirror))
+  )
   (gr_line (start 127.762 107.442) (end 127.762 96.774) (layer Edge.Cuts) (width 0.05))
