File: System_development/v0.2/PCB Design/Voltage_Regulator_v1/Voltage_Regulator_v2.kicad_pcb (KiCad board)
At the start: 2 copper layers, 35.6 x 19.8 mm, 5 parts, among them U1 LM7812_TO220

Commit message: Random
Routing:
- net GND: vias 4 -> 6
Other:
- board size 35.6 x 19.8 mm -> 35.6 x 24.1 mm
Changed lines of the file:
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@@
     )
   )
-  (gr_rect (start 157.48 98.552) (end 121.92 78.74) (layer "Edge.Cuts") (width 0.1) (fill none))
+  (gr_rect (start 157.48 101.4222) (end 121.92 77.2922) (layer "Edge.Cuts") (width 0.1) (fill none))
   (segment (start 135.28 91.44) (end 136.925 93.085) (width 0.25) (layer "F.Cu") (net 1))
   (segment (start 136.925 93.085) (end 136.925 94.674) (width 0.25) (layer "F.Cu") (net 1))
@@
   (segment (start 136.925 94.674) (end 135.079 96.52) (width 0.25) (layer "F.Cu") (net 1))
   (via (at 149.86 97.282) (size 0.8) (drill 0.4) (layers "F.Cu" "B.Cu") (free) (net 2))
+  (via (at 154.1272 80.0862) (size 0.8) (drill 0.4) (layers "F.Cu" "B.Cu") (free) (net 2))
   (via (at 128.778 97.282) (size 0.8) (drill 0.4) (layers "F.Cu" "B.Cu") (free) (net 2))
   (via (at 129.54 83.82) (size 0.8) (drill 0.4) (layers "F.Cu" "B.Cu") (free) (net 2))
+  (via (at 125.5268 80.264) (size 0.8) (drill 0.4) (layers "F.Cu" "B.Cu") (free) (net 2))
   (via (at 149.86 83.82) (size 0.8) (drill 0.4) (layers "F.Cu" "B.Cu") (free) (net 2))
   (segment (start 142.005 94.712) (end 143.813 96.52) (width 0.25) (layer "F.Cu") (net 3))
@@
     (polygon
       (pts
-        (xy 157.48 98.552)
-        (xy 121.92 98.552)
-        (xy 121.92 78.74)
-        (xy 157.48 78.74)
+        (xy 157.48 101.4222)
+        (xy 121.92 101.4222)
+        (xy 121.92 77.2922)
+        (xy 157.48 77.2922)
       )
     )
