File: System_development/v0.4/PCB Design/NMR Control Board V 0.4.1 - edited/NMR_Control_V0.4.1 - edited.kicad_pcb (KiCad board)
At the start: 2 copper layers, 139.7 x 88.9 mm, 57 parts

Commit message: Port name edits
Parts:
- renumbered 24V_DC1 to 24V_DC_IN, 24V_AMP1 to 24V_HP_AMP, F_OUT1 to F_OUT, Input1 to HP_AMP_IN, Impd_Match1 to Impd_Match, Output1 to LNA_IN, MIX_RF1 to MIXER_IN, PULSE_GEN_IN1 to PULSE_GEN_IN, SPL_IN1 to SPL_IN, TRIG_OUT1 to TRIG_OUT_1, SIN_SIGNAL_IN1 to TRIG_OUT_2
Changed lines of the file:
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@@
     (property "ki_keywords" "BNC SMA SMB SMC LEMO coaxial connector CINCH RCA")
     (attr smd)
-    (fp_text reference "SIN_SIGNAL_IN1" (at 0 -3.5) (layer "F.SilkS")
+    (fp_text reference "TRIG_OUT_2" (at 0 -3.5) (layer "F.SilkS")
         (effects (font (size 1 1) (thickness 0.15)))
     )
@@
     (property "ki_keywords" "BNC SMA SMB SMC LEMO coaxial connector CINCH RCA")
     (attr smd)
-    (fp_text reference "24V_DC1" (at 0.489 -3.809) (layer "F.SilkS")
+    (fp_text reference "24V_DC_IN" (at 0.489 -3.809) (layer "F.SilkS")
         (effects (font (size 1 1) (thickness 0.15)))
     )
@@
     (property "ki_keywords" "BNC SMA SMB SMC LEMO coaxial connector CINCH RCA")
     (attr through_hole)
-    (fp_text reference "MIX_RF1" (at 0 -4.75 90) (layer "F.SilkS")
+    (fp_text reference "MIXER_IN" (at 0 -4.75 90) (layer "F.SilkS")
         (effects (font (size 1 1) (thickness 0.15)))
     )
@@
     (property "ki_keywords" "BNC SMA SMB SMC LEMO coaxial connector CINCH RCA")
     (attr through_hole)
-    (fp_text reference "Impd_Match1" (at 0 -4.75) (layer "F.SilkS")
+    (fp_text reference "Impd_Match" (at 0 -4.75) (layer "F.SilkS")
         (effects (font (size 1 1) (thickness 0.15)))
     )
@@
     (property "ki_keywords" "BNC SMA SMB SMC LEMO coaxial connector CINCH RCA")
     (attr through_hole)
-    (fp_text reference "Output1" (at 0 -4.75 90) (layer "F.SilkS")
+    (fp_text reference "LNA_IN" (at 0 -4.75 90) (layer "F.SilkS")
         (effects (font (size 1 1) (thickness 0.15)))
     )
@@
     (property "ki_keywords" "BNC SMA SMB SMC LEMO coaxial connector CINCH RCA")
     (attr through_hole)
-    (fp_text reference "Input1" (at -0.0012 -4.9716) (layer "F.SilkS")
+    (fp_text reference "HP_AMP_IN" (at -0.0012 -4.9716) (layer "F.SilkS")
         (effects (font (size 1 1) (thickness 0.15)))
     )
@@
     (property "ki_keywords" "BNC SMA SMB SMC LEMO coaxial connector CINCH RCA")
     (attr smd)
-    (fp_text reference "SPL_IN1" (at 0 -3.5) (layer "F.SilkS")
+    (fp_text reference "SPL_IN" (at 0 -3.5) (layer "F.SilkS")
         (effects (font (size 1 1) (thickness 0.15)))
     )
@@
     (property "ki_keywords" "BNC SMA SMB SMC LEMO coaxial connector CINCH RCA")
     (attr through_hole)
-    (fp_text reference "24V_AMP1" (at 0.1412 5.142) (layer "F.SilkS")
+    (fp_text reference "24V_HP_AMP" (at 0.1412 5.142) (layer "F.SilkS")
         (effects (font (size 1 1) (thickness 0.15)))
     )
@@
     (property "ki_keywords" "BNC SMA SMB SMC LEMO coaxial connector CINCH RCA")
     (attr smd)
-    (fp_text reference "TRIG_OUT1" (at 0 -3.5) (layer "F.SilkS")
+    (fp_text reference "TRIG_OUT_1" (at 0 -3.5) (layer "F.SilkS")
         (effects (font (size 1 1) (thickness 0.15)))
     )
@@
     (property "ki_keywords" "BNC SMA SMB SMC LEMO coaxial connector CINCH RCA")
     (attr smd)
-    (fp_text reference "F_OUT1" (at 0 -3.5) (layer "F.SilkS")
+    (fp_text reference "F_OUT" (at 0 -3.5) (layer "F.SilkS")
         (effects (font (size 1 1) (thickness 0.15)))
     )
@@
     (property "ki_keywords" "BNC SMA SMB SMC LEMO coaxial connector CINCH RCA")
     (attr smd)
-    (fp_text reference "PULSE_GEN_IN1" (at 0 -3.5) (layer "F.SilkS")
-        (effects (font (size 1 1) (thickness 0.15)))
-    )
+    (fp_text reference "PULSE_GEN_IN" (at 0 -3.5) (layer "F.SilkS")
+        (effects (font (size 1 1) (thickness 0.15)))
+    )
