File: System_development/v0.5/PCB Design/NMR_ControlBoard_v0.5/NMR Control Board V 0.5.kicad_pcb (KiCad board)
At the start: 4 copper layers, 42 x 60 mm, 52 parts

Commit message: Edit NMR Control v0.5
Added two SMA connectors to RF switch input.
Parts:
- added SIN_SIGNAL_IN1: SIN_SIGNAL_IN1, Connector_Coaxial:SMA_Samtec_SMA-J-P-X-ST-EM1_EdgeMount, F.Cu at (66.0, 126.8)
- added TRIG_OUT1: TRIG_OUT1, Connector_Coaxial:SMA_Samtec_SMA-J-P-X-ST-EM1_EdgeMount, F.Cu at (60.2, 116.0)
- moved PG1 5.20 mm to (60.2, 107.5)
- moved SPL_IN1 5.00 mm to (75.0, 126.8)
- moved SW_OUT1 4.40 mm to (60.2, 99.1)
- moved D5 4.14 mm to (81.5, 118.2)
- moved D7 4.14 mm to (81.4, 121.7)
- moved MIX_RF1 3.70 mm to (60.3, 90.5)
- moved D6 3.69 mm to (86.3, 119.8), turned to -90 degrees
- moved OUTPUT1 3.65 mm to (84.0, 126.8)
- moved C8 3.10 mm to (74.6, 86.0)
- moved C6 2.97 mm to (64.6, 111.0)
- moved PWR_SPLITTER 2.97 mm to (67.3, 113.0)
- moved 1.8v_reg 2.95 mm to (65.8, 107.2)
- moved C13 2.95 mm to (64.2, 103.5)
- moved C5 2.95 mm to (66.7, 103.5)
- moved RF_SWITCH 2.95 mm to (65.6, 105.0)
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- renumbered -5v_REG to -5v_reg, 1.8v_REG to 1.8v_reg, 12v_REG to 12v_reg, 24_DC1 to 24V_DC1, 5v_REG to 5v_reg, PULSE_GEN_IN1 to PG1
Routing:
- net GND: track 178.3 -> 90.5 mm, vias 87 -> 70
- net Net-(J6-In): track 6.91 -> 30.7 mm
- net Net-(J5-In): track 8.64 -> 13.7 mm
- net Net-(D3-A): track 28.5 -> 24.3 mm
- net IF: track 3.98 -> 6.48 mm
- net 5v: track 39.7 -> 42.0 mm
- net Net-(J9-In): track 5.73 -> 6.66 mm
- net Net-(U5--IN1): track 8.36 -> 7.85 mm
Other:
- outline, holes or cut-outs redrawn
