File: System_development/v0.5/PCB Design/NMR_ControlBoard_v0.5/NMR Control Board V 0.5.kicad_sch (KiCad schematic)
At the start: 53 parts, among them J1 24V_AMP1, J10 INPUT1, J11 Z_MATCH1, J12 OUTPUT1, J2 24V_DC1, J3 F_OUT1, J4 MIX_RF1, J5 SPL_IN1, J6 PULSE_GEN_IN1, J7 SIN_SIGNAL_IN1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

Commit message: Edit NMR Control v0.5
Added two SMA connectors to RF switch input.
Connections:
- net GND: now also J6.2 (Ext), J7.2 (Ext), J8.2 (Ext), J9.2 (Ext), U8.3 (GND), U8.5 (GND), U8.6 (GND), U8.7 (GND)
Changed lines of the file:
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@@
+    (stroke (width 0) (type default))
+  )
+  (wire (pts (xy 49.784 181.864) (xy 49.784 183.134))
     (stroke (width 0) (type default))
   )
@@
         )
       )
+    )
+  )
+  (symbol (lib_id "power:GND") (at 49.784 183.134 0) (unit 1)
+    (in_bom yes) (on_board yes) (dnp no) (fields_autoplaced)
+    (property "Reference" "#PWR08" (at 49.784 189.484 0)
+      (effects (font (size 1.27 1.27)) hide)
+    )
+    (property "Value" "GND" (at 49.784 187.96 0)
+      (effects (font (size 1.27 1.27)))
+    )
+    (property "Footprint" "" (at 49.784 183.134 0)
+      (effects (font (size 1.27 1.27)) hide)
+    )
+    (property "Datasheet" "" (at 49.784 183.134 0)
+      (effects (font (size 1.27 1.27)) hide)
+    )
+    (pin "1")
+    (instances
+      (project "NMR Control Board V 0.5"
+        (path "/1de478d9-4249-4d6f-b43f-fd31039cff25"
+          (reference "#PWR08") (unit 1)
+        )
+      )
