File: System_development/Van-Hove/PCB Design/NMR Control Board V 0.4.2/PCB Design.kicad_pcb (KiCad board)
At the start: 2 copper layers, 139 x 89 mm, 58 parts

Commit message: Add files via upload
Parts:
- removed ? (x3): , 
- added TP1: TestPoint, TestPoint:TestPoint_Keystone_5000-5004_Miniature, F.Cu at (133.0, 109.5)
- added TP10: TestPoint, TestPoint:TestPoint_Keystone_5000-5004_Miniature, F.Cu at (168.5, 74.5)
- added TP11: TestPoint, TestPoint:TestPoint_Keystone_5000-5004_Miniature, F.Cu at (185.5, 109.5)
- added TP12: TestPoint, TestPoint:TestPoint_Keystone_5000-5004_Miniature, F.Cu at (179.0, 117.5)
- added TP13: TestPoint, TestPoint:TestPoint_Keystone_5000-5004_Miniature, F.Cu at (191.5, 126.0)
- added TP14: TestPoint, TestPoint:TestPoint_Keystone_5000-5004_Miniature, F.Cu at (201.0, 88.5)
- added TP15: TestPoint, TestPoint:TestPoint_Keystone_5000-5004_Miniature, F.Cu at (189.0, 100.0)
- added TP16: TestPoint, TestPoint:TestPoint_Keystone_5000-5004_Miniature, F.Cu at (105.0, 84.0)
- added TP17: TestPoint, TestPoint:TestPoint_Keystone_5000-5004_Miniature, F.Cu at (126.0, 91.0)
- added TP18: TestPoint, TestPoint:TestPoint_Keystone_5000-5004_Miniature, F.Cu at (134.5, 97.0)
- added TP2: TestPoint, TestPoint:TestPoint_Keystone_5000-5004_Miniature, F.Cu at (178.5, 82.0)
- added TP3: TestPoint, TestPoint:TestPoint_Keystone_5000-5004_Miniature, F.Cu at (146.5, 96.0)
- added TP4: TestPoint, TestPoint:TestPoint_Keystone_5000-5004_Miniature, F.Cu at (147.5, 100.0)
- added TP5: TestPoint, TestPoint:TestPoint_Keystone_5000-5004_Miniature, F.Cu at (145.0, 75.5)
- added TP6: TestPoint, TestPoint:TestPoint_Keystone_5000-5004_Miniature, F.Cu at (110.5, 82.5)
- added TP7: TestPoint, TestPoint:TestPoint_Keystone_5000-5004_Miniature, F.Cu at (136.0, 83.5)
- added TP8: TestPoint, TestPoint:TestPoint_Keystone_5000-5004_Miniature, F.Cu at (192.0, 87.5)
- added TP9: TestPoint, TestPoint:TestPoint_Keystone_5000-5004_Miniature, F.Cu at (166.0, 119.0)
- -5V_REG1: footprint VanHove:Mf05A -> V 0.4.2 Footprints:Mf05A
- 1.8V_Reg.1: footprint VanHove:1.8VReg -> V 0.4.2 Footprints:1.8VReg
- 12V_REG1: footprint VanHove:5VReg -> V 0.4.2 Footprints:5VReg
- 5V_REG1: footprint VanHove:5VReg2 -> V 0.4.2 Footprints:5VReg2
- C1, C10, C11, C12, C13, C14, C15, C2, C3, C4, C5, C6, C7, C8, C9, R1, R2, R3, R4: footprint VanHove:CustomR -> V 0.4.2 Footprints:CustomR
- J1: renamed from IMPED MATCH
- J10: renamed from SINE IN; footprint Connector_Coaxial:SMA_Samtec_SMA-J-P-X-ST-EM1_EdgeMount -> Connector_Coaxial:SMA_Amphenol_132134_Vertical
- J11: renamed from MIXER IN
- J12: renamed from F_OUT; footprint Connector_Coaxial:SMA_Samtec_SMA-J-P-X-ST-EM1_EdgeMount -> Connector_Coaxial:SMA_Amphenol_132134_Vertical
- J2: renamed from HP AMP IN
- J3: renamed from LNA IN
- J4: renamed from Pulse_Gen_In; footprint Connector_Coaxial:SMA_Samtec_SMA-J-P-X-ST-EM1_EdgeMount -> Connector_Coaxial:SMA_Amphenol_132134_Vertical
- J5: renamed from 24V HP AMP
- J6: renamed from 24V DC IN; footprint Connector_Coaxial:SMA_Samtec_SMA-J-P-X-ST-EM1_EdgeMount -> Connector_Coaxial:SMA_Amphenol_132134_Vertical
- J7: renamed from SINE TRIG; footprint Connector_Coaxial:SMA_Samtec_SMA-J-P-X-ST-EM1_EdgeMount -> Connector_Coaxial:SMA_Amphenol_132134_Vertical
- J8: renamed from TRIG_OUT; footprint Connector_Coaxial:SMA_Samtec_SMA-J-P-X-ST-EM1_EdgeMount -> Connector_Coaxial:SMA_Amphenol_132134_Vertical
- J9: renamed from SINE OUT
- LNA1: footprint VanHove:LNA -> V 0.4.2 Footprints:LNA
- Mixer1: footprint VanHove:Mixer2 -> V 0.4.2 Footprints:Mixer2
- PWRSplitter1: footprint VanHove:Mini-Circuits_CD636_LandPatternPL-035 -> V 0.4.2 Footprints:Mini-Circuits_CD636_LandPatternPL-035
- REF** (x4): value MountingHole_3.2mm_M3_ISO7380_Pad -> Mount
- Switch1: footprint VanHove:Switch -> V 0.4.2 Footprints:Switch
- moved C10 50.0 mm to (135.5, 102.8), turned to 90 degrees
- moved C12 50.0 mm to (183.4, 88.5), turned to 0 degrees
- moved C4 45.9 mm to (169.0, 109.8)
- moved C8 45.9 mm to (123.3, 114.5)
- moved C13 15.8 mm to (146.4, 82.5)
- moved C14 15.8 mm to (162.2, 82.8)
- moved G*** 11.0 mm to (151.0, 97.5)
- moved G*** 6.18 mm to (117.5, 76.5)
- moved J6 2.84 mm to (107.0, 145.5)
- moved J10 1.50 mm to (185.5, 67.5)
- moved J12 1.50 mm to (141.7, 67.5)
- moved J4 1.50 mm to (123.8, 67.5)
- moved J7 1.50 mm to (208.0, 67.5)
- moved J8 1.50 mm to (163.7, 67.5)
- moved C7 0.50 mm to (155.5, 137.8)
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Connections:
- C10 pad 1: Net-(1.8V_Reg.1-OUT) -> Net-(-5V_REG1-V+)
- C12 pad 1: Net-(-5V_REG1-V+) -> Net-(1.8V_Reg.1-OUT)
- C13 pad 1: GND -> Net-(LNA1-+IN1)
- C13 pad 2: Net-(J12-In) -> Net-(Mixer1-IF)
- C14 pad 1: Net-(LNA1-+IN1) -> GND
- C14 pad 2: Net-(Mixer1-IF) -> Net-(J12-In)
- C4 pad 1: Net-(+12VPin1-In) -> Net-(1.8V_Reg.1-OUT)
- C8 pad 1: Net-(1.8V_Reg.1-OUT) -> Net-(+12VPin1-In)
- R1 pad 1: Net-(LNA1--IN1) -> Net-(LNA1-OUT1)
- R1 pad 2: Net-(LNA1-OUT1) -> Net-(LNA1--IN1)
- R3 pad 1: GND -> Net-(LNA1--IN1)
- R3 pad 2: Net-(LNA1--IN1) -> GND
Routing:
- net Net-(-5V_REG1-C1-): track 13.5 -> 32.4 mm, vias 1 -> 0
- net Net-(LNA1--IN1): track 17.1 -> 31.3 mm, vias 1 -> 0
- net Net-(1.8V_Reg.1-OUT): track 37.7 -> 51.3 mm, vias 1 -> 0
- net GND: track 22.2 -> 33.5 mm, vias 53 -> 160
- net Net-(J11-In): track 89.2 -> 79.8 mm, vias 1 -> 0
- net Net-(J4-In): track 135.1 -> 143.7 mm
- net Net-(Mixer1-LO): track 32.8 -> 40.3 mm, vias 3 -> 2
- net Net-(-5V_REG1-C1+): track 9.21 -> 16.5 mm, vias 1 -> 0
- net Net-(J9-In): track 31.6 -> 38.1 mm, vias 3 -> 2
- net Net-(-5V_REG1-V+): track 97.9 -> 104.2 mm, vias 1 -> 0
- net Net-(LNA1-+IN1): track 16.0 -> 21.3 mm, vias 1 -> 0
- net Net-(J10-In): track 50.0 -> 54.9 mm, vias 1 -> 0
- net Net-(-5V_REG1-OUT): track 49.6 -> 53.5 mm, vias 1 -> 0
- net Net-(Mixer1-IF): track 60.2 -> 63.7 mm
- net Net-(+12VPin1-In): track 151.1 -> 149.1 mm
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Other:
- board text added: "-5V Regulator"
- board text added: "1.8V Regulator"
- board text added: "12V Regulator"
- board text added: "5V Regulator"
- board text removed: "-5V Reg"
- board text removed: "1.8V Reg"
- board text removed: "12V Reg"
- board text removed: "5V Reg"
- board text removed: "P"
