File: System_development/Van-Hove/PCB Design/NMR Control Board V 0.4.2/PCB Design.kicad_sch (KiCad schematic)
At the start: 49 parts, among them J1 Imped Match, J10 SPI In, J11 Mix RF, J12 Output Function, J2 Input 1, J3 Output, J4 Pulse Wave, J5 24V Amp, J6 24V DC, J7 Sine Wave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

Commit message: Add files via upload
Parts:
- added TP1, TP10, TP11, TP12, TP13, TP14, TP15, TP16, TP17, TP18, TP2, TP3, TP4, TP5, TP6, TP7, TP8, TP9: TestPoint, TestPoint:TestPoint_Keystone_5000-5004_Miniature, symbol Connector:TestPoint
- -5V_REG1: footprint VanHove:Mf05A -> V 0.4.2 Footprints:Mf05A
- 1.8V_Reg.1: footprint VanHove:1.8VReg -> V 0.4.2 Footprints:1.8VReg
- 12V_REG1: footprint VanHove:5VReg -> V 0.4.2 Footprints:5VReg
- 5V_REG1: footprint VanHove:5VReg2 -> V 0.4.2 Footprints:5VReg2
- C1, C10, C11, C12, C13, C14, C15, C2, C3, C4, C5, C6, C7, C8, C9, R1, R2, R3, R4: footprint VanHove:CustomR -> V 0.4.2 Footprints:CustomR
- J10, J12, J4, J6, J7, J8: footprint Connector_Coaxial:SMA_Samtec_SMA-J-P-X-ST-EM1_EdgeMount -> Connector_Coaxial:SMA_Amphenol_132134_Vertical
- LNA1: footprint VanHove:LNA -> V 0.4.2 Footprints:LNA
- Mixer1: footprint VanHove:Mixer2 -> V 0.4.2 Footprints:Mixer2
- PWRSplitter1: footprint VanHove:Mini-Circuits_CD636_LandPatternPL-035 -> V 0.4.2 Footprints:Mini-Circuits_CD636_LandPatternPL-035
- Switch1: footprint VanHove:Switch -> V 0.4.2 Footprints:Switch
Connections:
- net GND: now also C14.1, J10.2 (Ext), J11.2 (Ext), J2.2 (Ext), J4.2 (Ext), J5.2 (Ext), J6.2 (Ext), J7.2 (Ext), J8.2 (Ext), R3.2; no longer C14.2, J10.1 (In), J11.1 (In), J2.1 (In), J4.1 (In), J5.1 (In), J6.1 (In), J7.1 (In), J8.1 (In), R3.1
- net at -5V_REG1.2 (V+), 1.8V_Reg.1.4 (IN), 5V_REG1.2 (VO)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: now also TP1.1, TP4.1
- net at 1.8V_Reg.1.5 (OUT), C12.1, C4.1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: now also TP2.1, TP9.1
- net at D1.1 (K), D2.2 (A): now also J2.1 (In); no longer J2.2 (Ext)
- net at J12.1 (In), R2.2: now also C14.2; no longer C14.1
- net at LNA1.1 (OUT1), R2.1: now also R1.1, TP3.1; no longer R1.2
- net at 12V_REG1.1 (VI), C5.1: now also J5.1 (In), J6.1 (In); no longer J5.2 (Ext), J6.2 (Ext)
- net at C13.1, LNA1.3 (+IN1), R4.1: now also TP7.1
- net at J9.1 (In), Switch1.8 (RF2): now also TP8.1
- net at Mixer1.3 (RF): now also J11.1 (In), TP13.1; no longer J11.2 (Ext)
- net at PWRSplitter1.1 (SUM): now also J10.1 (In), TP14.1; no longer J10.2 (Ext)
- net at Mixer1.6 (LO), PWRSplitter1.3 (PORT1): now also TP11.1
- net at PWRSplitter1.4 (PORT2), Switch1.4 (RF1): now also TP15.1
- net at -5V_REG1.1 (OUT), C11.1, C3.1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: now also TP16.1, TP6.1
- net at -5V_REG1.3 (C1-), C2.2: now also TP18.1
- net at -5V_REG1.5 (C1+), C2.1: now also TP17.1
- net at C13.2, Mixer1.2 (IF): now also TP12.1
- new net: LNA1.2 (-IN1), R1.2, R3.1, TP5.1
- new net: J4.1 (In), J7.1 (In), J8.1 (In), Switch1.2 (CTRL), TP10.1
Other:
- moved on the sheet: C14, J10, J11, J2, J4, J5, J6, J7, J8, R1, R3
