File: System_development/Van-Hove/PCB_design/NMR Control Board V 0.4.4/PCB Design.kicad_pcb (KiCad board)
At the start: 2 copper layers, 139 x 89 mm, 75 parts

Commit message: Readme File Changed
Other:
- board text added: "NMR Control V 0.4.4 Jake Martin Angelo Varillas Winford Usman Khan Daniel Hancock Josh Hager"
- board text removed: "NMR Control V 0.4.4 Jake Martin Angelo Varillas Winford Janvrin Daniel Hancock Asifuzzaman Khan Josh Hager"
Changed lines of the file:
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@@
 		)
 	)
-	(gr_text "NMR Control V 0.4.4\nJake Martin\nAngelo Varillas\nWinford Janvrin\nDaniel Hancock\nAsifuzzaman Khan\nJosh Hager"
+	(gr_text "NMR Control V 0.4.4\nJake Martin\nAngelo Varillas\nWinford\nUsman Khan \nDaniel Hancock\nJosh Hager"
 		(at 108 74.5 0)
 		(layer "F.SilkS")
