File: System_development/Van-Hove/PCB_design/Impedance Matching Board v0.2/impedance matching.kicad_pcb (KiCad board)
At the start: 2 copper layers, 10.4 x 40.8 mm, 4 parts, among them J1 Conn_Coaxial, J2 Conn_Coaxial

Commit message: fixed version number spacing, adding logos/QR code to coil connector.
Other:
- board text added: "Impedence Matching Board v0.2"
- board text removed: "Impedence Matching Board V0.2"
Changed lines of the file:
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@@
 	)
 	(paper "A4")
+	(title_block
+		(title "NMR Impedance Matching Board")
+		(date "2026-04-01")
+		(rev "v0.2")
+	)
 	(layers
 		(0 "F.Cu" signal)
@@
 		(layer "Edge.Cuts")
 	)
-	(gr_text "Impedence Matching Board V0.2"
+	(gr_text "Impedence Matching Board v0.2"
 		(at 148.5 115 270)
 		(layer "B.SilkS")
