File: System_development/Van-Hove/PCB_design/NMR Control Board v0.4.5/PCB Design.kicad_sch (KiCad schematic)
At the start: 68 parts, among them J1 Imped Match, J10 SPI In, J11 Mix RF, J12 Output Function, J2 Input 1, J3 Output, J4 Pulse Wave, J5 24V Amp, J6 24V DC, J7 Sine Wave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

Commit message: Updated BoM
Parts:
- C6: value C14 -> ~
- C7: value C15 -> ~
- L1: value L -> 0.56 μH
Changed lines of the file:
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@@
 			)
 		)
-		(property "Datasheet" " ~"
+		(property "Datasheet" "~"
 			(at 17.78 170.18 0)
 			(effects
@@
 			)
 		)
-		(property "Datasheet" " ~"
+		(property "Datasheet" "~"
 			(at 182.88 158.75 0)
 			(effects
@@
 			)
 		)
-		(property "Value" "C15"
+		(property "Value" "~"
 			(at 100.33 172.7199 0)
 			(effects
@@
 			)
 		)
-		(property "Datasheet" " ~"
+		(property "Datasheet" "~"
 			(at 120.65 49.53 0)
 			(effects
@@
 			)
 		)
-		(property "Datasheet" " ~"
+		(property "Datasheet" "~"
 			(at 149.86 90.17 0)
 			(effects
@@
 			)
 		)
-		(property "Datasheet" " ~"
+		(property "Datasheet" "~"
 			(at 200.66 77.47 0)
 			(effects
@@
 			)
 		)
-		(property "Datasheet" " ~"
+		(property "Datasheet" "~"
 			(at 15.24 132.08 0)
 			(effects
@@
 			)
 		)
-		(property "Datasheet" " ~"
+		(property "Datasheet" "~"
 			(at 166.37 31.75 0)
 			(effects
@@
 			)
 		)
-		(property "Datasheet" " ~"
+		(property "Datasheet" "~"
 			(at 125.73 96.52 0)
 			(effects
@@
 			)
 		)
-		(property "Datasheet" " ~"
+		(property "Datasheet" "~"
 			(at 74.93 132.08 0)
 			(effects
@@
 			)
 		)
-		(property "Datasheet" " ~"
+		(property "Datasheet" "~"
 			(at 88.9 125.73 0)
 			(effects
@@
 			)
 		)
-		(property "Value" "L"
+		(property "Value" "0.56 μH"
 			(at 87.63 165.1 90)
 			(effects
@@
 			)
 		)
-		(property "Datasheet" " ~"
+		(property "Datasheet" "~"
 			(at 27.94 132.08 0)
 			(effects
@@
 			)
 		)
-		(property "Datasheet" " ~"
+		(property "Datasheet" "~"
 			(at 57.15 168.91 0)
 			(effects
@@
 			)
 		)
-		(property "Datasheet" " ~"
+		(property "Datasheet" "~"
 			(at 132.08 81.28 0)
 			(effects
@@
 			)
 		)
-		(property "Datasheet" " ~"
+		(property "Datasheet" "~"
 			(at 133.35 50.8 0)
 			(effects
@@
 			)
 		)
-		(property "Value" "C14"
+		(property "Value" "~"
 			(at 80.01 172.7199 0)
 			(effects
